File: zusi interface/zusi interface/zusi interface.kicad_pcb (KiCad board)
At the start: 2 copper layers, 17 parts, among them CON1 TAGconnect, J1 Conn_01x02, U1 PCF8574A, U2 ESP32-WROOM

Commit message: prop dev
aan mijn prop dev board getekend
Parts:
- added C1: C_Small, Resistor_SMD:R_0402_1005Metric, F.Cu at (157.7, 57.4)
- added C2: C_Small, Resistor_SMD:R_0402_1005Metric, F.Cu at (149.6, 79.1)
- added C3: C_Small, Resistor_SMD:R_0402_1005Metric, F.Cu at (149.7, 77.6)
- added C4: C_Small, Resistor_SMD:R_0402_1005Metric, F.Cu at (160.3, 57.3)
- added C5: C_Small, Resistor_SMD:R_0402_1005Metric, F.Cu at (144.3, 67.8)
- added C6: C_Small, Resistor_SMD:R_0402_1005Metric, F.Cu at (144.3, 66.7)
- added D3: LED_Small_ALT, LED_SMD:LED_0402_1005Metric, F.Cu at (202.4, 60.0)
- added D4: LED_Small_ALT, LED_SMD:LED_0402_1005Metric, F.Cu at (202.4, 58.9)
- added D5: LED_Small_ALT, LED_SMD:LED_0402_1005Metric, F.Cu at (192.3, 57.4)
- added D6: LED_Small_ALT, LED_SMD:LED_0402_1005Metric, F.Cu at (192.3, 58.7)
- added D7: LED_Small_ALT, LED_SMD:LED_0402_1005Metric, F.Cu at (192.3, 59.9)
- added D8: LED_Small_ALT, LED_SMD:LED_0402_1005Metric, F.Cu at (157.7, 68.9)
- added D9: LED_Small_ALT, LED_SMD:LED_0402_1005Metric, F.Cu at (157.7, 67.5)
- added RN1: R_Network07, Resistor_THT:R_Array_SIP8, F.Cu at (210.0, 74.4)
- added U3: NCP1117ST33T3G, Package_TO_SOT_SMD:SOT-223, F.Cu at (144.9, 74.0)
- D1, D2: value LTST-C191TBKT -> LED_Small_ALT; footprint Diode_SMD:D_0402_1005Metric -> LED_SMD:LED_0402_1005Metric
- R4: footprint Inductor_SMD:L_0603_1608Metric -> Inductor_SMD:L_0402_1005Metric
- moved JP1 170.8 mm to (208.4, 58.7), turned to 270 degrees
- moved U1 154.5 mm to (197.2, 61.9)
- moved D1 149.6 mm to (202.3, 62.4)
- moved JP2 146.3 mm to (208.6, 64.0), turned to 90 degrees
- moved U2 146.1 mm to (171.6, 62.7)
- moved JP3 142.7 mm to (205.0, 68.7)
- moved D2 133.6 mm to (202.3, 61.3)
- moved R5 122.2 mm to (183.0, 74.4), turned to 270 degrees
- moved R7 116.5 mm to (191.5, 64.1), turned to 270 degrees
- moved R6 114.6 mm to (192.8, 65.8), turned to 270 degrees
- moved R1 107.2 mm to (192.7, 61.9), turned to 270 degrees
- moved R2 99.2 mm to (159.9, 68.9), turned to 180 degrees
- moved R3 97.0 mm to (160.0, 67.5), turned to 180 degrees
- moved CON1 94.3 mm to (177.4, 81.1), turned to 180 degrees
- moved BZ1 93.5 mm to (159.9, 81.1), turned to 270 degrees
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Connections:
- D1 pad 1: +3V3 -> Net-(D1-Pad1)
- D2 pad 1: +3V3 -> Net-(D2-Pad1)
- J1 pad 1: Net-(J1-Pad1) -> GND
- J1 pad 2: +3V3 -> +12V
- R2 pad 2: Net-(D1-Pad2) -> Net-(D8-Pad2)
- R3 pad 2: Net-(D2-Pad2) -> Net-(D9-Pad2)
- U1 pad 4: Net-(U1-Pad4) -> Net-(D1-Pad1)
- U1 pad 5: Net-(U1-Pad5) -> Net-(D2-Pad1)
- U2 pad 11: /~int -> Net-(U2-Pad11)
- U2 pad 33: Net-(U2-Pad33) -> /~int
Routing:
- net +3V3: track 0.00 -> 180.4 mm
- net GND: track 0.00 -> 78.2 mm, vias 0 -> 43
- net /Enable: track 0.00 -> 36.1 mm
- net Net-(D5-Pad2): track 0.00 -> 27.8 mm, vias 0 -> 1
- net /RX: track 0.00 -> 26.8 mm, vias 0 -> 3
- net Net-(D6-Pad2): track 0.00 -> 26.3 mm, vias 0 -> 1
- net Net-(D7-Pad2): track 0.00 -> 22.2 mm, vias 0 -> 1
- net /GPIO0: track 0.00 -> 22.1 mm, vias 0 -> 2
- net /TX: track 0.00 -> 21.2 mm, vias 0 -> 2
- net Net-(D4-Pad2): track 0.00 -> 20.7 mm, vias 0 -> 1
- net Net-(D3-Pad2): track 0.00 -> 19.8 mm, vias 0 -> 1
- net /SDA: track 0.00 -> 17.6 mm, vias 0 -> 3
- net Net-(D2-Pad2): track 0.00 -> 16.3 mm, vias 0 -> 1
- net /SCL: track 0.00 -> 16.1 mm, vias 0 -> 2
- net Net-(D1-Pad2): track 0.00 -> 15.7 mm, vias 0 -> 1
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- added copper zone on B.Cu, net GND
Other:
- board outline added: 86.4 x 36.6 mm
- net class Default: via_dia 0.8 -> 0.6; via_drill 0.4 -> 0.3
- rule via_min_size: 0.4 -> 0.6
- board text added: "+"
- board text added: "Ontworpen door Ben De Lathouwer V0"
- board text added: "Zusi pzb en AWI interface"
