File: zusi interface/zusi interface/zusi interface.sch (KiCad schematic (older format))
At the start: 17 parts, among them CON1 TAGconnect, J1 Conn_01x02, U1 PCF8574A, U2 ESP32-WROOM

Commit message: prop dev
aan mijn prop dev board getekend
Parts:
- removed D1, D2: LTST-C191TBKT, Diode_SMD:D_0402_1005Metric, symbol dk_LED-Indication-Discrete:LTST-C191TBKT
- added C1, C2, C3, C4, C5, C6: C_Small, Resistor_SMD:R_0402_1005Metric, symbol Device:C_Small
- added D1, D2, D3, D4, D5, D6, D7, D8, D9: LED_Small_ALT, LED_SMD:LED_0402_1005Metric, symbol Device:LED_Small_ALT
- added RN1: R_Network07, Resistor_THT:R_Array_SIP8, symbol Device:R_Network07
- added U3: NCP1117ST33T3G, Package_TO_SOT_SMD:SOT-223, symbol dk_PMIC-Voltage-Regulators-Linear:NCP1117ST33T3G
Connections:
- net labels added: +12V
- wire segments 90 -> 131
Other:
- note added: "I2C port expander\n"
- note added: "Voeding en ontkopeling \n"
- note added: "Wifi+Programming \n"
