File: propellor dev/propellor dev board/propellor dev board.sch (KiCad schematic (older format))
At the start: 2 parts

Commit message: pcb done
pcb afgetekend voor propellor dev board
Parts:
- added C3, C5: 10u, Capacitor_THT:CP_Radial_D10.0mm_P3.80mm, symbol Device:C_Small
- added C4, C6: 100n, Capacitor_THT:C_Rect_L7.0mm_W3.5mm_P2.50mm_P5.00mm, symbol Device:C_Small
- added D1: 1N4007, Diode_THT:D_DO-41_SOD81_P10.16mm_Horizontal, symbol Diode:1N4007
- added J1: 2pin header, Connector_PinHeader_2.54mm:PinHeader_1x02_P2.54mm_Vertical, symbol Connector_Generic:Conn_01x02
- added J2, J3: Conn_01x16_Male, Connector_PinSocket_2.54mm:PinSocket_1x16_P2.54mm_Vertical, symbol Connector:Conn_01x16_Male
- added J4: Conn_01x06, Connector_PinSocket_2.54mm:PinSocket_1x06_P2.54mm_Vertical, symbol Connector_Generic:Conn_01x06
- added R1: 10K, Resistor_THT:R_Axial_DIN0207_L6.3mm_D2.5mm_P15.24mm_Horizontal, symbol Device:R_Small
- added U1: propstick, Connector_PinHeader_2.54mm:PinHeader_1x04_P2.54mm_Vertical, symbol programmers:propstick
- added U2: LM7805_TO220, Package_TO_SOT_THT:TO-220-3_Vertical, symbol Regulator_Linear:LM7805_TO220
- added U3: LM1117-3.3, Package_TO_SOT_THT:TO-220-3_Vertical, symbol Regulator_Linear:LM1117-3.3
- added U4: 24LC256, Package_DIP:DIP-8_W7.62mm_LongPads, symbol Memory_EEPROM:24LC256
- gave numbers to parts that had none: 2
Connections:
- net labels added: +5V, SCL, SDA, VAA
- wire segments 24 -> 109
