File: propellor dev/propellor dev board/propellor dev board.kicad_pcb (KiCad board)
At the start: 2 copper layers, 102.9 x 101.6 mm, 16 parts, among them J1 2pin header, J2 Conn_01x16_Male, J3 Conn_01x16_Male, J4 Conn_01x06, U1 propstick, U2 LM7805_TO220, U3 LM1117-3.3, U4 24LC256, U5 P8X32A-D40, Y1 Crystal_Small

Commit message: af
3d body's beginnen toevoegen
Parts:
- added REF**: KiCad-Logo2_12mm_SilkScreen, Symbol:KiCad-Logo2_12mm_SilkScreen, F.Cu at (173.0, 32.1)
- added REF**: OSHW-Symbol_13.4x12mm_SilkScreen, Symbol:OSHW-Symbol_13.4x12mm_SilkScreen, F.Cu at (194.8, 33.2)
- added REF**: Fiducial_1mm_Dia_2mm_Outer, Fiducial:Fiducial_1mm_Dia_2mm_Outer, F.Cu at (103.4, 28.8)
- added REF**: Fiducial_1mm_Dia_2mm_Outer, Fiducial:Fiducial_1mm_Dia_2mm_Outer, F.Cu at (102.6, 124.9)
- added REF**: Fiducial_1mm_Dia_2mm_Outer, Fiducial:Fiducial_1mm_Dia_2mm_Outer, F.Cu at (199.8, 124.5)
Other:
- board text added: "by Ben De Lathouwer"
